Commit message: Removed redundant transmissions created my moveit setup assistant

File: add_post_pro_simulation/urdf/add_post_pro_robot.urdf.xacro (robot description, xacro)
@@ -699,4 +699,5 @@
         </sensor>
     </gazebo>
+    <!-- END OF SCANCONTROL -->
     <gazebo reference="EEF_sensor_holder">
         <material>Gazebo/CoM</material>
@@ -705,853 +706,3 @@
         <material>Gazebo/CoM</material>
     </gazebo>
-    <transmission name="trans_joint_1">
-        <type>transmission_interface/SimpleTransmission</type>
-        <joint name="joint_1">
-            <hardwareInterface>hardware_interface/EffortJointInterface</hardwareInterface>
-        </joint>
-        <actuator name="joint_1_motor">
-            <hardwareInterface>hardware_interface/EffortJointInterface</hardwareInterface>
-            <mechanicalReduction>1</mechanicalReduction>
-        </actuator>
-    </transmission>
-    <transmission name="trans_joint_2">
-        <type>transmission_interface/SimpleTransmission</type>
-        <joint name="joint_2">
-            <hardwareInterface>hardware_interface/EffortJointInterface</hardwareInterface>
-        </joint>
-        <actuator name="joint_2_motor">
-            <hardwareInterface>hardware_interface/EffortJointInterface</hardwareInterface>
-            <mechanicalReduction>1</mechanicalReduction>
-        </actuator>
-    </transmission>
-    <transmission name="trans_joint_3">
-        <type>transmission_interface/SimpleTransmission</type>
-        <joint name="joint_3">
-            <hardwareInterface>hardware_interface/EffortJointInterface</hardwareInterface>
-        </joint>
-        <actuator name="joint_3_motor">
-            <hardwareInterface>hardware_interface/EffortJointInterface</hardwareInterface>
-            <mechanicalReduction>1</mechanicalReduction>
-        </actuator>
-    </transmission>
-    <transmission name="trans_joint_4">
-        <type>transmission_interface/SimpleTransmission</type>
-        <joint name="joint_4">
-            <hardwareInterface>hardware_interface/EffortJointInterface</hardwareInterface>
-        </joint>
-        <actuator name="joint_4_motor">
-            <hardwareInterface>hardware_interface/EffortJointInterface</hardwareInterface>
-            <mechanicalReduction>1</mechanicalReduction>
-        </actuator>
-    </transmission>
-    <transmission name="trans_joint_5">
-        <type>transmission_interface/SimpleTransmission</type>
-        <joint name="joint_5">
-            <hardwareInterface>hardware_interface/EffortJointInterface</hardwareInterface>
-        </joint>
-        <actuator name="joint_5_motor">
-            <hardwareInterface>hardware_interface/EffortJointInterface</hardwareInterface>
-            <mechanicalReduction>1</mechanicalReduction>
-        </actuator>
-    </transmission>
-    <transmission name="trans_joint_6">
-        <type>transmission_interface/SimpleTransmission</type>
-        <joint name="joint_6">
-            <hardwareInterface>hardware_interface/EffortJointInterface</hardwareInterface>
-        </joint>
-        <actuator name="joint_6_motor">
-            <hardwareInterface>hardware_interface/EffortJointInterface</hardwareInterface>
-            <mechanicalReduction>1</mechanicalReduction>
-        </actuator>
-    </transmission>
-    <transmission name="trans_turntable_revolve_joint">
-        <type>transmission_interface/SimpleTransmission</type>
-        <joint name="turntable_revolve_joint">
-            <hardwareInterface>hardware_interface/EffortJointInterface</hardwareInterface>
-        </joint>
-        <actuator name="turntable_revolve_joint_motor">
-            <hardwareInterface>hardware_interface/EffortJointInterface</hardwareInterface>
-            <mechanicalReduction>1</mechanicalReduction>
-        </actuator>
-    </transmission>
-    <gazebo>
-        <plugin name="gazebo_ros_control" filename="libgazebo_ros_control.so">
-            <robotNamespace>/</robotNamespace>
-        </plugin>
-    </gazebo>
-    <transmission name="trans_1">
-        <type>transmission_interface/SimpleTransmission</type>
-        <joint name="joint_1">
-            <hardwareInterface>hardware_interface/PositionJointInterface</hardwareInterface>
-        </joint>
-        <actuator name="motor_1">
-            <hardwareInterface>hardware_interface/PositionJointInterface</hardwareInterface>
-            <mechanicalReduction>1</mechanicalReduction>
-        </actuator>
-    </transmission>
-    <transmission name="trans_2">
-        <type>transmission_interface/SimpleTransmission</type>
-        <joint name="joint_2">
-            <hardwareInterface>hardware_interface/PositionJointInterface</hardwareInterface>
-        </joint>
-        <actuator name="motor_2">
-            <hardwareInterface>hardware_interface/PositionJointInterface</hardwareInterface>
-            <mechanicalReduction>1</mechanicalReduction>
-        </actuator>
-    </transmission>
-    <transmission name="trans_3">
-        <type>transmission_interface/SimpleTransmission</type>
-        <joint name="joint_3">
-            <hardwareInterface>hardware_interface/PositionJointInterface</hardwareInterface>
-        </joint>
-        <actuator name="motor_3">
-            <hardwareInterface>hardware_interface/PositionJointInterface</hardwareInterface>
-            <mechanicalReduction>1</mechanicalReduction>
-        </actuator>
-    </transmission>
-    <transmission name="trans_4">
-        <type>transmission_interface/SimpleTransmission</type>
-        <joint name="joint_4">
-            <hardwareInterface>hardware_interface/PositionJointInterface</hardwareInterface>
-        </joint>
-        <actuator name="motor_4">
-            <hardwareInterface>hardware_interface/PositionJointInterface</hardwareInterface>
-            <mechanicalReduction>1</mechanicalReduction>
-        </actuator>
-    </transmission>
-    <transmission name="trans_5">
-        <type>transmission_interface/SimpleTransmission</type>
-        <joint name="joint_5">
-            <hardwareInterface>hardware_interface/PositionJointInterface</hardwareInterface>
-        </joint>
-        <actuator name="motor_5">
-            <hardwareInterface>hardware_interface/PositionJointInterface</hardwareInterface>
-            <mechanicalReduction>1</mechanicalReduction>
-        </actuator>
-    </transmission>
-    <transmission name="trans_6">
-        <type>transmission_interface/SimpleTransmission</type>
-        <joint name="joint_6">
-            <hardwareInterface>hardware_interface/PositionJointInterface</hardwareInterface>
-        </joint>
-        <actuator name="motor_6">
-            <hardwareInterface>hardware_interface/PositionJointInterface</hardwareInterface>
-            <mechanicalReduction>1</mechanicalReduction>
-        </actuator>
-    </transmission>
-    <gazebo>
-        <plugin filename="libgazebo_ros_control.so" name="gazebo_ros_control">
-            <robotNamespace>/vs6577</robotNamespace>
-            <legacyModeNS>true</legacyModeNS>
-        </plugin>
-    </gazebo>
-    <link name="world" />
-    <joint name="joint_w" type="fixed">
-        <parent link="world" />
-        <child link="base_link" />
-        <origin xyz="0 0 0" />
-    </joint>
-    <link name="base_link">
-        <visual>
-            <origin rpy="0 0 0" xyz="0 0 0" />
-            <geometry>
-                <mesh filename="package://denso_robot_descriptions/vs6577_description/meshes/base_link.dae" scale="1 1 1" />
-            </geometry>
-        </visual>
-        <collision>
-            <origin rpy="0 0 0" xyz="0 0 0" />
-            <geometry>
-                <mesh filename="package://denso_robot_descriptions/vs6577_description/meshes/base_link.dae" scale="1 1 1" />
-            </geometry>
-        </collision>
-        <inertial>
-            <mass value="1" />
-            <origin rpy="0.000000 0.000000 0.000000" xyz="0.000000 0.000000 0.000000" />
-            <inertia ixx="1" ixy="0" ixz="0" iyy="1" iyz="0" izz="1" />
-        </inertial>
-    </link>
-    <link name="J1">
-        <visual>
-            <origin rpy="0 0 0" xyz="0 0 0" />
-            <geometry>
-                <mesh filename="package://denso_robot_descriptions/vs6577_description/meshes/J1.dae" scale="1 1 1" />
-            </geometry>
-        </visual>
-        <collision>
-            <origin rpy="0 0 0" xyz="0 0 0" />
-            <geometry>
-                <mesh filename="package://denso_robot_descriptions/vs6577_description/meshes/J1.dae" scale="1 1 1" />
-            </geometry>
-        </collision>
-        <inertial>
-            <mass value="1" />
-            <origin rpy="0.000000 0.000000 0.000000" xyz="0.000000 0.000000 0.000000" />
-            <inertia ixx="1" ixy="0" ixz="0" iyy="1" iyz="0" izz="1" />
-        </inertial>
-    </link>
-    <link name="J2">
-        <visual>
-            <origin rpy="0 0 0" xyz="0 0 0" />
-            <geometry>
-                <mesh filename="package://denso_robot_descriptions/vs6577_description/meshes/J2.dae" scale="1 1 1" />
-            </geometry>
-        </visual>
-        <collision>
-            <origin rpy="0 0 0" xyz="0 0 0" />
-            <geometry>
-                <mesh filename="package://denso_robot_descriptions/vs6577_description/meshes/J2.dae" scale="1 1 1" />
-            </geometry>
-        </collision>
-        <inertial>
-            <mass value="1" />
-            <origin rpy="0.000000 0.000000 0.000000" xyz="0.000000 0.000000 0.000000" />
-            <inertia ixx="1" ixy="0" ixz="0" iyy="1" iyz="0" izz="1" />
-        </inertial>
-    </link>
-    <link name="J3">
-        <visual>
-            <origin rpy="0 0 0" xyz="0 0 0" />
-            <geometry>
-                <mesh filename="package://denso_robot_descriptions/vs6577_description/meshes/J3.dae" scale="1 1 1" />
-            </geometry>
-        </visual>
-        <collision>
-            <origin rpy="0 0 0" xyz="0 0 0" />
-            <geometry>
-                <mesh filename="package://denso_robot_descriptions/vs6577_description/meshes/J3.dae" scale="1 1 1" />
-            </geometry>
-        </collision>
-        <inertial>
-            <mass value="1" />
-            <origin rpy="0.000000 0.000000 0.000000" xyz="0.000000 0.000000 0.000000" />
-            <inertia ixx="1" ixy="0" ixz="0" iyy="1" iyz="0" izz="1" />
-        </inertial>
-    </link>
-    <link name="J4">
-        <visual>
-            <origin rpy="0 0 0" xyz="0 0 0" />
-            <geometry>
-                <mesh filename="package://denso_robot_descriptions/vs6577_description/meshes/J4.dae" scale="1 1 1" />
-            </geometry>
-        </visual>
-        <collision>
-            <origin rpy="0 0 0" xyz="0 0 0" />
-            <geometry>
-                <mesh filename="package://denso_robot_descriptions/vs6577_description/meshes/J4.dae" scale="1 1 1" />
-            </geometry>
-        </collision>
-        <inertial>
-            <mass value="1" />
-            <origin rpy="0.000000 0.000000 0.000000" xyz="0.000000 0.000000 0.000000" />
-            <inertia ixx="1" ixy="0" ixz="0" iyy="1" iyz="0" izz="1" />
-        </inertial>
-    </link>
-    <link name="J5">
-        <visual>
-            <origin rpy="0 0 0" xyz="0 0 0" />
-            <geometry>
-                <mesh filename="package://denso_robot_descriptions/vs6577_description/meshes/J5.dae" scale="1 1 1" />
-            </geometry>
-        </visual>
-        <collision>
-            <origin rpy="0 0 0" xyz="0 0 0" />
-            <geometry>
-                <mesh filename="package://denso_robot_descriptions/vs6577_description/meshes/J5.dae" scale="1 1 1" />
-            </geometry>
-        </collision>
-        <inertial>
-            <mass value="1" />
-            <origin rpy="0.000000 0.000000 0.000000" xyz="0.000000 0.000000 0.000000" />
-            <inertia ixx="1" ixy="0" ixz="0" iyy="1" iyz="0" izz="1" />
-        </inertial>
-    </link>
-    <link name="J6">
-        <visual>
-            <origin rpy="0 0 0" xyz="0 0 0" />
-            <geometry>
-                <mesh filename="package://denso_robot_descriptions/vs6577_description/meshes/J6.dae" scale="1 1 1" />
-            </geometry>
-        </visual>
-        <collision>
-            <origin rpy="0 0 0" xyz="0 0 0" />
-            <geometry>
-                <mesh filename="package://denso_robot_descriptions/vs6577_description/meshes/J6.dae" scale="1 1 1" />
-            </geometry>
-        </collision>
-        <inertial>
-            <mass value="1" />
-            <origin rpy="0.000000 0.000000 0.000000" xyz="0.000000 0.000000 0.000000" />
-            <inertia ixx="1" ixy="0" ixz="0" iyy="1" iyz="0" izz="1" />
-        </inertial>
-    </link>
-    <gazebo reference="base_link">
-        <material>Gazebo/CoM</material>
-    </gazebo>
-    <gazebo reference="J1">
-        <material>Gazebo/Gray</material>
-    </gazebo>
-    <gazebo reference="J2">
-        <material>Gazebo/Gray</material>
-    </gazebo>
-    <gazebo reference="J3">
-        <material>Gazebo/Gray</material>
-    </gazebo>
-    <gazebo reference="J4">
-        <material>Gazebo/Gray</material>
-    </gazebo>
-    <gazebo reference="J5">
-        <material>Gazebo/Gray</material>
-    </gazebo>
-    <gazebo reference="J6">
-        <material>Gazebo/Gray</material>
-    </gazebo>
-    <gazebo reference="EEF_tool_mount">
-        <material>Gazebo/CoM</material>
-    </gazebo>
-    <gazebo>
-        <gravity>False</gravity>
-    </gazebo>
-    <joint name="joint_1" type="revolute">
-        <parent link="base_link" />
-        <child link="J1" />
-        <origin rpy="0.000000 0.000000 0.000000" xyz="0.000000 0.000000 0.000000" />
-        <axis xyz="-0.000000 -0.000000 1.000000" />
-        <limit effort="100" lower="-2.96706" upper="2.96706" velocity="1" />
-        <dynamics damping="0" friction="0" />
-    </joint>
-    <joint name="joint_2" type="revolute">
-        <parent link="J1" />
-        <child link="J2" />
-        <origin rpy="0.000000 0.000000 0.000000" xyz="0.075000 0.000000 0.335000" />
-        <axis xyz="-0.000000 1.000000 -0.000000" />
-        <limit effort="100" lower="-1.745329" upper="2.356194" velocity="1" />
-        <dynamics damping="0" friction="0" />
-    </joint>
-    <joint name="joint_3" type="revolute">
-        <parent link="J2" />
-        <child link="J3" />
-        <origin rpy="0.000000 0.000000 0.000000" xyz="0.000000 0.000000 0.365000" />
-        <axis xyz="-0.000000 1.000000 -0.000000" />
-        <limit effort="100" lower="-2.076942" upper="2.949606" velocity="1" />
-        <dynamics damping="0" friction="0" />
-    </joint>
-    <joint name="joint_4" type="revolute">
-        <parent link="J3" />
-        <child link="J4" />
-        <origin rpy="0.000000 0.000000 0.000000" xyz="-0.090000 0.000000 -0.700000" />
-        <axis xyz="-0.000000 -0.000000 1.000000" />
-        <limit effort="100" lower="-3.316126" upper="3.316126" velocity="1" />
-        <dynamics damping="0" friction="0" />
-    </joint>
-    <joint name="joint_5" type="revolute">
-        <parent link="J4" />
-        <child link="J5" />
-        <origin rpy="0.000000 0.000000 0.000000" xyz="0.000000 0.000000 1.105000" />
-        <axis xyz="-0.000000 1.000000 -0.000000" />
-        <limit effort="100" lower="-2.094395" upper="2.094395" velocity="1" />
-        <dynamics damping="0" friction="0" />
-    </joint>
-    <joint name="joint_6" type="revolute">
-        <parent link="J5" />
-        <child link="J6" />
-        <origin rpy="0.000000 0.000000 0.000000" xyz="0.000000 0.000000 0.080000" />
-        <axis xyz="-0.000000 -0.000000 1.000000" />
-        <limit effort="100" lower="-6.283185" upper="6.283185" velocity="1" />
-        <dynamics damping="0" friction="0" />
-    </joint>
-    <link name="turntable_base">
-        <visual>
-            <origin rpy="0 0 0" xyz="0 0 0" />
-            <geometry>
-                <cylinder length=".32" radius=".02" />
-            </geometry>
-        </visual>
-        <collision>
-            <origin rpy="0 0 0" xyz="0 0 0" />
-            <geometry>
-                <cylinder length=".32" radius=".02" />
-            </geometry>
-        </collision>
-        <inertial>
-            <origin rpy="0 0 0" xyz="0 0 0" />
-            <mass value="1" />
-            <inertia ixx="100" ixy="0" ixz="0" iyy="100" iyz="0" izz="100" />
-        </inertial>
-    </link>
-    <link name="turntable_plate">
-        <visual>
-            <origin rpy="0 0 0" xyz="0 0 0" />
-            <geometry>
-                <cylinder length=".01" radius=".15" />
-            </geometry>
-            <material name="Red">
-                <color rgba="1.0 0 0 1.0" />
-            </material>
-        </visual>
-        <collision>
-            <origin rpy="0 0 0" xyz="0 0 0" />
-            <geometry>
-                <cylinder length=".01" radius=".15" />
-            </geometry>
-        </collision>
-        <inertial>
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